File: Electronics/Control Board/Control Board.sch (EAGLE design)
At the start: 0 parts

Commit message: Added filler for control module and flushed out body sketch some more. Added two more displays
Parts:
- added JP1, JP2: M10-M20-9991046, Control Board Library:M10-M20-9991046
- added STANDOFF1, STANDOFF2, STANDOFF3, STANDOFF4: STAND-OFF, Resistor Module Library:STAND-OFF
Connections:
- new net 5V: JP1.6
- new net 5V_2: JP2.6
- new net EEPROM_CS_L: JP1.1
- new net EEPROM_MISO: JP1.4
- new net EEPROM_MOSI: JP1.2
- new net EEPROM_SCK: JP1.3
- new net GND: JP1.5
- new net GND_2: JP2.5
- new net R_IN: JP2.1
- new net R_OUT: JP2.2
- new net SERIAL_CLK: JP1.8
- new net SERIAL_CLK_2: JP2.8
- new net SERIAL_IN: JP2.4
- new net SERIAL_LATCH: JP1.9
- new net SERIAL_LATCH_2: JP2.9
- new net SERIAL_MR_L: JP1.7
- new net SERIAL_MR_L_2: JP2.7
- new net SERIAL_OE_L: JP1.10
- new net SERIAL_OE_L_2: JP2.10
