File: Electronics/Control Board/Control Board.sch (EAGLE design)
At the start: 6 parts

Commit message: Started work on control board.
Connections:
- net SERIAL_IN renamed SERIAL_OUT
- removed net 5V_2: JP2.6
- removed net GND_2: JP2.5
- removed net SERIAL_CLK_2: JP2.8
- removed net SERIAL_LATCH_2: JP2.9
- removed net SERIAL_MR_L_2: JP2.7
- removed net SERIAL_OE_L_2: JP2.10
- net 5V: now also JP2.6
- net GND: now also JP2.5
- net R_IN: now also JP2.2; no longer JP2.1
- net R_OUT: now also JP2.1; no longer JP2.2
- net SERIAL_CLK: now also JP2.8
- net SERIAL_LATCH: now also JP2.9
- net SERIAL_MR_L: now also JP2.7
- net SERIAL_OE_L: now also JP2.10
Changed lines of the file:
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@@
 </variantdefs>
 <classes>
-<class number="0" name="default" width="0" drill="0">
+<class number="0" name="default" width="0.2032" drill="0.4064">
+<clearance class="0" value="0.2032"/>
+</class>
+<class number="1" name="power" width="0.6096" drill="0.4064">
+<clearance class="1" value="0.2032"/>
+</class>
+<class number="2" name="gnd" width="0.3048" drill="0.4064">
+<clearance class="2" value="0.2032"/>
+</class>
+<class number="3" name="power usb" width="0.508" drill="0.4064">
+<clearance class="3" value="0.2032"/>
 </class>
 </classes>
@@
 <part name="SUPPLY6" library="Resistor Module Library" deviceset="5V" device=""/>
 <part name="GND19" library="Resistor Module Library" deviceset="DGND" device=""/>
+<part name="GND1" library="Resistor Module Library" deviceset="DGND" device=""/>
+<part name="SUPPLY1" library="Resistor Module Library" deviceset="5V" device=""/>
 </parts>
 <sheets>
 <sheet>
+<description>Mechanical</description>
 <plain>
 </plain>
@@
 </sheet>
 <sheet>
+<description>Interface</description>
 <plain>
 </plain>
@@
 <instance part="SUPPLY6" gate="G$1" x="35.56" y="5.08"/>
 <instance part="GND19" gate="G$1" x="35.56" y="-7.62"/>
+<instance part="GND1" gate="G$1" x="106.68" y="-5.08"/>
+<instance part="SUPPLY1" gate="G$1" x="106.68" y="0"/>
 </instances>
 <busses>
@@
 <pinref part="JP1" gate="G$1" pin="9"/>
 </segment>
+<segment>
+<wire x1="83.82" y1="7.62" x2="101.6" y2="7.62" width="0.1524" layer="91"/>
+<label x="83.82" y="7.62" size="1.778" layer="95"/>
+<pinref part="JP2" gate="G$1" pin="9"/>
+</segment>
 </net>
 <net name="SERIAL_OE_L" class="0">
@@
 <label x="7.62" y="10.16" size="1.778" layer="95"/>
 <pinref part="JP1" gate="G$1" pin="10"/>
+</segment>
+<segment>
+<wire x1="83.82" y1="10.16" x2="104.14" y2="10.16" width="0.1524" layer="91"/>
+<label x="83.82" y="10.16" size="1.778" layer="95"/>
+<pinref part="JP2" gate="G$1" pin="10"/>
 </segment>
 </net>
@@
 <pinref part="SUPPLY6" gate="G$1" pin="5V"/>
 </segment>
+<segment>
+<pinref part="JP2" gate="G$1" pin="6"/>
+<wire x1="83.82" y1="0" x2="106.68" y2="0" width="0.1524" layer="91"/>
+<label x="93.98" y="0" size="1.778" layer="95"/>
+<pinref part="SUPPLY1" gate="G$1" pin="5V"/>
+<junction x="106.68" y="0"/>
+</segment>
 </net>
 <net name="GND" class="0">
@@
 <pinref part="GND19" gate="G$1" pin="GND"/>
 </segment>
+<segment>
+<pinref part="JP2" gate="G$1" pin="5"/>
+<wire x1="83.82" y1="-2.54" x2="106.68" y2="-2.54" width="0.1524" layer="91"/>
+<label x="93.98" y="-2.54" size="1.778" layer="95"/>
+<pinref part="GND1" gate="G$1" pin="GND"/>
+<junction x="106.68" y="-2.54"/>
+</segment>
 </net>
-<net name="SERIAL_IN" class="0">
+<net name="SERIAL_OUT" class="0">
 <segment>
 <pinref part="JP2" gate="G$1" pin="4"/>
 <wire x1="83.82" y1="-5.08" x2="99.06" y2="-5.08" width="0.1524" layer="91"/>
 <label x="86.36" y="-5.08" size="1.778" layer="95"/>
-</segment>
-</net>
-<net name="SERIAL_OE_L_2" class="0">
-<segment>
-<wire x1="83.82" y1="10.16" x2="104.14" y2="10.16" width="0.1524" layer="91"/>
-<label x="83.82" y="10.16" size="1.778" layer="95"/>
-<pinref part="JP2" gate="G$1" pin="10"/>
-</segment>
-</net>
-<net name="SERIAL_LATCH_2" class="0">
-<segment>
-<wire x1="83.82" y1="7.62" x2="101.6" y2="7.62" width="0.1524" layer="91"/>
-<label x="83.82" y="7.62" size="1.778" layer="95"/>
-<pinref part="JP2" gate="G$1" pin="9"/>
-</segment>
-</net>
-<net name="5V_2" class="0">
-<segment>
-<pinref part="JP2" gate="G$1" pin="6"/>
-<wire x1="83.82" y1="0" x2="111.76" y2="0" width="0.1524" layer="91"/>
-<label x="93.98" y="0" size="1.778" layer="95"/>
-</segment>
-</net>
-<net name="GND_2" class="0">
-<segment>
-<pinref part="JP2" gate="G$1" pin="5"/>
-<wire x1="83.82" y1="-2.54" x2="111.76" y2="-2.54" width="0.1524" layer="91"/>
-<label x="93.98" y="-2.54" size="1.778" layer="95"/>
 </segment>
 </net>
@@
 </net>
 <net name="R_IN" class="0">
-<segment>
-<pinref part="JP2" gate="G$1" pin="1"/>
-<wire x1="83.82" y1="-12.7" x2="99.06" y2="-12.7" width="0.1524" layer="91"/>
-<label x="86.36" y="-12.7" size="1.778" layer="95"/>
-</segment>
-</net>
-<net name="R_OUT" class="0">
 <segment>
 <pinref part="JP2" gate="G$1" pin="2"/>
@@
 <pinref part="JP1" gate="G$1" pin="7"/>
 </segment>
-</net>
-<net name="SERIAL_MR_L_2" class="0">
 <segment>
 <wire x1="104.14" y1="2.54" x2="83.82" y2="2.54" width="0.1524" layer="91"/>
@@
 <pinref part="JP1" gate="G$1" pin="8"/>
 </segment>
-</net>
-<net name="SERIAL_CLK_2" class="0">
 <segment>
 <wire x1="101.6" y1="5.08" x2="83.82" y2="5.08" width="0.1524" layer="91"/>
@@
 </segment>
 </net>
+<net name="R_OUT" class="0">
+<segment>
+<pinref part="JP2" gate="G$1" pin="1"/>
+<wire x1="83.82" y1="-12.7" x2="99.06" y2="-12.7" width="0.1524" layer="91"/>
+<label x="86.36" y="-12.7" size="1.778" layer="95"/>
+</segment>
+</net>
 </nets>
 </sheet>
+<sheet>
+<plain>
+</plain>
+<instances>
+</instances>
+<busses>
+</busses>
+<nets>
+</nets>
+</sheet>

Commit message: Selected 8U2 microchip for main controller. Don't need a lot of IO and needed included USB drive
Parts:
- added U1: ATMEGA8U2AU, Control Board Library:ATMEGA8U2AU
Connections:
- net 5V: now also U1.AVCC, U1.VCC
- net GND: now also U1.GND, U1.UGND
Changed lines of the file:
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@@
 <part name="GND1" library="Resistor Module Library" deviceset="DGND" device=""/>
 <part name="SUPPLY1" library="Resistor Module Library" deviceset="5V" device=""/>
+<part name="U1" library="Control Board Library" deviceset="ATMEGA8U2" device="AU"/>
+<part name="GND2" library="Control Board Library" deviceset="DGND" device=""/>
+<part name="SUPPLY2" library="Control Board Library" deviceset="5V" device=""/>
 </parts>
 <sheets>
@@
 </plain>
 <instances>
+<instance part="U1" gate="G$1" x="0" y="0"/>
+<instance part="GND2" gate="G$1" x="-25.4" y="-33.02"/>
+<instance part="SUPPLY2" gate="G$1" x="-25.4" y="22.86"/>
 </instances>
 <busses>
 </busses>
 <nets>
+<net name="5V" class="0">
+<segment>
+<pinref part="SUPPLY2" gate="G$1" pin="5V"/>
+<pinref part="U1" gate="G$1" pin="VCC"/>
+<wire x1="-25.4" y1="22.86" x2="-20.32" y2="22.86" width="0.1524" layer="91"/>
+<pinref part="U1" gate="G$1" pin="AVCC"/>
+<wire x1="-20.32" y1="22.86" x2="-20.32" y2="20.32" width="0.1524" layer="91"/>
+<junction x="-20.32" y="22.86"/>
+</segment>
+</net>
+<net name="GND" class="0">
+<segment>
+<pinref part="U1" gate="G$1" pin="GND"/>
+<pinref part="GND2" gate="G$1" pin="GND"/>
+<wire x1="-20.32" y1="-27.94" x2="-25.4" y2="-27.94" width="0.1524" layer="91"/>
+<wire x1="-25.4" y1="-27.94" x2="-25.4" y2="-30.48" width="0.1524" layer="91"/>
+<pinref part="U1" gate="G$1" pin="UGND"/>
+<wire x1="-20.32" y1="-27.94" x2="-20.32" y2="-25.4" width="0.1524" layer="91"/>
+<junction x="-20.32" y="-27.94"/>
+</segment>
+</net>
 </nets>
 </sheet>
